Commit message: fix: initialize Stage4 Gazebo joints from YAML home
Co-authored-by: Cursor <cursoragent@cursor.com>

File: src/fairino3_gazebo/urdf/fairino3_gazebo.urdf.xacro (robot description, xacro)
@@ -14,4 +14,11 @@
   <xacro:arg name="world_to_base_pitch" default="0"/>
   <xacro:arg name="world_to_base_yaw" default="0"/>
+  <!-- Stage 1–3 defaults match the previous hardcoded Gazebo pose. -->
+  <xacro:arg name="initial_j1" default="0.8377"/>
+  <xacro:arg name="initial_j2" default="-1.1927"/>
+  <xacro:arg name="initial_j3" default="1.1129"/>
+  <xacro:arg name="initial_j4" default="-1.1499"/>
+  <xacro:arg name="initial_j5" default="-3.1393"/>
+  <xacro:arg name="initial_j6" default="2.0996"/>
   <!-- FAIRINO 官方 FR3 -->
   <xacro:include
@@ -37,5 +44,11 @@
   <xacro:include
       filename="$(find fairino3_gazebo)/urdf/gz_ros2_control.xacro"/>
-  <xacro:fr3_gz_ros2_control/>
+  <xacro:fr3_gz_ros2_control
+      initial_j1="$(arg initial_j1)"
+      initial_j2="$(arg initial_j2)"
+      initial_j3="$(arg initial_j3)"
+      initial_j4="$(arg initial_j4)"
+      initial_j5="$(arg initial_j5)"
+      initial_j6="$(arg initial_j6)"/>
   <!-- gz_ros2_control Gazebo Plugin -->
   <gazebo>

File: src/fairino3_gazebo/urdf/gz_ros2_control.xacro (robot description, xacro)
@@ -1,5 +1,7 @@
 <?xml version="1.0"?>
 <robot xmlns:xacro="http://www.ros.org/wiki/xacro">
-  <xacro:macro name="fr3_gz_ros2_control">
+  <!-- Defaults keep Stage 1–3 / generic sim pose unchanged. Stage 4 overrides. -->
+  <xacro:macro name="fr3_gz_ros2_control"
+      params="initial_j1:=0.8377 initial_j2:=-1.1927 initial_j3:=1.1129 initial_j4:=-1.1499 initial_j5:=-3.1393 initial_j6:=2.0996">
     <ros2_control
         name="GazeboSimSystem"
@@ -12,5 +14,5 @@
         <state_interface name="position">
           <param name="initial_value">
-            0.8377
+            ${initial_j1}
           </param>
         </state_interface>
@@ -21,5 +23,5 @@
         <state_interface name="position">
           <param name="initial_value">
-            -1.1927
+            ${initial_j2}
           </param>
         </state_interface>
@@ -30,5 +32,5 @@
         <state_interface name="position">
           <param name="initial_value">
-            1.1129
+            ${initial_j3}
           </param>
         </state_interface>
@@ -39,5 +41,5 @@
         <state_interface name="position">
           <param name="initial_value">
-            -1.1499
+            ${initial_j4}
           </param>
         </state_interface>
@@ -48,5 +50,5 @@
         <state_interface name="position">
           <param name="initial_value">
-            -3.1393
+            ${initial_j5}
           </param>
         </state_interface>
@@ -57,5 +59,5 @@
         <state_interface name="position">
           <param name="initial_value">
-            2.0996
+            ${initial_j6}
           </param>
         </state_interface>
